File: KeyboardPCB/KeyboardPCB.kicad_sch (KiCad schematic)
At the start: 0 parts

Commit message: added some diodes
Other:
- sheet Key_Array ports: added ICOL0, ICOL1, ICOL10, ICOL11, ICOL12, ICOL13, ICOL14, ICOL15, ICOL2, ICOL3, ICOL4, ICOL5, ICOL6, ICOL7, ICOL8, ICOL9; removed none
- sheet MCU_Battery ports: added COL0, COL1; removed none
Changed lines of the file:
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@@
 (kicad_sch (version 20211123) (generator eeschema)
   (paper "A4")
+  (wire (pts (xy 139.7 77.47) (xy 152.4 77.47))
+    (stroke (width 0) (type default) (color 0 0 0 0))
+  )
+  (wire (pts (xy 139.7 62.23) (xy 152.4 62.23))
+    (stroke (width 0) (type default) (color 0 0 0 0))
+  )
   (wire (pts (xy 139.7 129.54) (xy 152.4 129.54))
     (stroke (width 0) (type default) (color 0 0 0 0))
   )
+  (wire (pts (xy 139.7 80.01) (xy 152.4 80.01))
+    (stroke (width 0) (type default) (color 0 0 0 0))
+  )
+  (wire (pts (xy 139.7 64.77) (xy 152.4 64.77))
+    (stroke (width 0) (type default) (color 0 0 0 0))
+  )
+  (wire (pts (xy 139.7 72.39) (xy 152.4 72.39))
+    (stroke (width 0) (type default) (color 0 0 0 0))
+  )
+  (wire (pts (xy 139.7 57.15) (xy 152.4 57.15))
+    (stroke (width 0) (type default) (color 0 0 0 0))
+  )
+  (wire (pts (xy 139.7 69.85) (xy 152.4 69.85))
+    (stroke (width 0) (type default) (color 0 0 0 0))
+  )
+  (wire (pts (xy 139.7 46.99) (xy 152.4 46.99))
+    (stroke (width 0) (type default) (color 0 0 0 0))
+  )
   (wire (pts (xy 139.7 127) (xy 152.4 127))
     (stroke (width 0) (type default) (color 0 0 0 0))
   )
+  (wire (pts (xy 139.7 82.55) (xy 152.4 82.55))
+    (stroke (width 0) (type default) (color 0 0 0 0))
+  )
+  (wire (pts (xy 139.7 44.45) (xy 152.4 44.45))
+    (stroke (width 0) (type default) (color 0 0 0 0))
+  )
   (wire (pts (xy 139.7 134.62) (xy 152.4 134.62))
     (stroke (width 0) (type default) (color 0 0 0 0))
@@
   )
   (wire (pts (xy 139.7 124.46) (xy 152.4 124.46))
+    (stroke (width 0) (type default) (color 0 0 0 0))
+  )
+  (wire (pts (xy 139.7 49.53) (xy 152.4 49.53))
+    (stroke (width 0) (type default) (color 0 0 0 0))
+  )
+  (wire (pts (xy 139.7 54.61) (xy 152.4 54.61))
+    (stroke (width 0) (type default) (color 0 0 0 0))
+  )
+  (wire (pts (xy 139.7 74.93) (xy 152.4 74.93))
+    (stroke (width 0) (type default) (color 0 0 0 0))
+  )
+  (wire (pts (xy 139.7 52.07) (xy 152.4 52.07))
+    (stroke (width 0) (type default) (color 0 0 0 0))
+  )
+  (wire (pts (xy 139.7 59.69) (xy 152.4 59.69))
+    (stroke (width 0) (type default) (color 0 0 0 0))
+  )
+  (wire (pts (xy 139.7 67.31) (xy 152.4 67.31))
     (stroke (width 0) (type default) (color 0 0 0 0))
   )
@@
       (effects (font (size 1.27 1.27)) (justify right))
     )
+    (pin "COL1" input (at 139.7 46.99 0)
+      (effects (font (size 1.27 1.27)) (justify right))
+    )
+    (pin "COL0" input (at 139.7 44.45 0)
+      (effects (font (size 1.27 1.27)) (justify right))
+    )
   )
   (sheet (at 152.4 25.4) (size 114.3 114.3) (fields_autoplaced)
@@
       (effects (font (size 1.27 1.27)) (justify left))
     )
+    (pin "ICOL9" input (at 152.4 67.31 180)
+      (effects (font (size 1.27 1.27)) (justify left))
+    )
+    (pin "ICOL8" input (at 152.4 64.77 180)
+      (effects (font (size 1.27 1.27)) (justify left))
+    )
+    (pin "ICOL0" input (at 152.4 44.45 180)
+      (effects (font (size 1.27 1.27)) (justify left))
+    )
+    (pin "ICOL14" input (at 152.4 80.01 180)
+      (effects (font (size 1.27 1.27)) (justify left))
+    )
+    (pin "ICOL15" input (at 152.4 82.55 180)
+      (effects (font (size 1.27 1.27)) (justify left))
+    )
+    (pin "ICOL12" input (at 152.4 74.93 180)
+      (effects (font (size 1.27 1.27)) (justify left))
+    )
+    (pin "ICOL10" input (at 152.4 69.85 180)
+      (effects (font (size 1.27 1.27)) (justify left))
+    )
+    (pin "ICOL11" input (at 152.4 72.39 180)
+      (effects (font (size 1.27 1.27)) (justify left))
+    )
+    (pin "ICOL13" input (at 152.4 77.47 180)
+      (effects (font (size 1.27 1.27)) (justify left))
+    )
+    (pin "ICOL3" input (at 152.4 52.07 180)
+      (effects (font (size 1.27 1.27)) (justify left))
+    )
+    (pin "ICOL1" input (at 152.4 46.99 180)
+      (effects (font (size 1.27 1.27)) (justify left))
+    )
+    (pin "ICOL2" input (at 152.4 49.53 180)
+      (effects (font (size 1.27 1.27)) (justify left))
+    )
+    (pin "ICOL4" input (at 152.4 54.61 180)
+      (effects (font (size 1.27 1.27)) (justify left))
+    )
+    (pin "ICOL5" input (at 152.4 57.15 180)
+      (effects (font (size 1.27 1.27)) (justify left))
+    )
+    (pin "ICOL6" input (at 152.4 59.69 180)
+      (effects (font (size 1.27 1.27)) (justify left))
+    )
+    (pin "ICOL7" input (at 152.4 62.23 180)
+      (effects (font (size 1.27 1.27)) (justify left))
+    )
   )
   (sheet_instances
@@
       (reference "#PWR?") (unit 1) (value "GND") (footprint "")
     )
-    (path "/0e04ce72-6533-49cc-b4b5-6fa7ba1a6887/ac8c0548-9166-47ec-a85f-139f0e9a6d98"
-      (reference "#PWR?") (unit 1) (value "GND") (footprint "")
-    )
     (path "/0e04ce72-6533-49cc-b4b5-6fa7ba1a6887/afce16ac-5064-4d84-8271-858b78925b08"
       (reference "#PWR?") (unit 1) (value "GND") (footprint "")
@@
     (path "/0e04ce72-6533-49cc-b4b5-6fa7ba1a6887/f72b91bb-4963-49bc-9a06-44650fc96a66"
       (reference "#PWR?") (unit 1) (value "GND") (footprint "")
-    )
-    (path "/0e04ce72-6533-49cc-b4b5-6fa7ba1a6887/280f704d-840e-4a66-a435-b638c5d9233f"
-      (reference "C?") (unit 1) (value "C") (footprint "")
     )
     (path "/0e04ce72-6533-49cc-b4b5-6fa7ba1a6887/8c980024-088c-474b-904a-257356022afa"
       (reference "C?") (unit 1) (value "C") (footprint "")
     )
-    (path "/0e04ce72-6533-49cc-b4b5-6fa7ba1a6887/ae40d9b4-7939-4535-bc5f-605681edeac5"
-      (reference "C?") (unit 1) (value "C") (footprint "")
-    )
     (path "/0e04ce72-6533-49cc-b4b5-6fa7ba1a6887/baf55504-1638-4b06-86e0-17fd16d0a675"
       (reference "C?") (unit 1) (value "C") (footprint "")
@@
       (reference "D?") (unit 1) (value "1N4148WT") (footprint "Diode_SMD:D_SOD-523")
     )
+    (path "/ea7fdac0-4451-48b5-bbfd-e0f47d60ba04/38fde887-7f04-44cc-88cf-f6af2cd6408f"
+      (reference "D?") (unit 1) (value "1N4148WT") (footprint "Diode_SMD:D_SOD-523")
+    )
     (path "/ea7fdac0-4451-48b5-bbfd-e0f47d60ba04/41cf5a6e-7eaf-4a99-af9a-7c6d950a495f"
       (reference "D?") (unit 1) (value "1N4148WT") (footprint "Diode_SMD:D_SOD-523")
@@
       (reference "D?") (unit 1) (value "1N4148WT") (footprint "Diode_SMD:D_SOD-523")
     )
+    (path "/ea7fdac0-4451-48b5-bbfd-e0f47d60ba04/4daa9c11-46fc-4755-8fbb-5cf894f357aa"
+      (reference "D?") (unit 1) (value "1N4148WT") (footprint "Diode_SMD:D_SOD-523")
+    )
     (path "/ea7fdac0-4451-48b5-bbfd-e0f47d60ba04/501e12a6-9a36-4baf-80f5-810ca392bffd"
       (reference "D?") (unit 1) (value "1N4148WT") (footprint "Diode_SMD:D_SOD-523")
@@
       (reference "D?") (unit 1) (value "1N4148WT") (footprint "Diode_SMD:D_SOD-523")
     )
+    (path "/ea7fdac0-4451-48b5-bbfd-e0f47d60ba04/90dfd895-6926-43ca-92f7-04222f754217"
+      (reference "D?") (unit 1) (value "1N4148WT") (footprint "Diode_SMD:D_SOD-523")
+    )
     (path "/ea7fdac0-4451-48b5-bbfd-e0f47d60ba04/92a1e4cf-9acd-481f-b88e-e8b9a265ecdf"
       (reference "D?") (unit 1) (value "1N4148WT") (footprint "Diode_SMD:D_SOD-523")
@@
       (reference "D?") (unit 1) (value "1N4148WT") (footprint "Diode_SMD:D_SOD-523")
     )
+    (path "/ea7fdac0-4451-48b5-bbfd-e0f47d60ba04/9b314d72-f022-4800-a87a-0262cd7678cd"
+      (reference "D?") (unit 1) (value "1N4148WT") (footprint "Diode_SMD:D_SOD-523")
+    )
     (path "/ea7fdac0-4451-48b5-bbfd-e0f47d60ba04/a85d7478-307e-47f5-a60f-3f2421d1bcea"
       (reference "D?") (unit 1) (value "1N4148WT") (footprint "Diode_SMD:D_SOD-523")
     )
+    (path "/ea7fdac0-4451-48b5-bbfd-e0f47d60ba04/bae01162-fa18-413f-bdbe-3d42a37a0ad3"
+      (reference "D?") (unit 1) (value "1N4148WT") (footprint "Diode_SMD:D_SOD-523")
+    )
     (path "/ea7fdac0-4451-48b5-bbfd-e0f47d60ba04/d176cf6e-56df-4a40-b93b-80e097893c73"
       (reference "D?") (unit 1) (value "1N4148WT") (footprint "Diode_SMD:D_SOD-523")
@@
     )
     (path "/ea7fdac0-4451-48b5-bbfd-e0f47d60ba04/f54334f0-73c8-4d3f-8db3-1519a520ddd0"
+      (reference "D?") (unit 1) (value "1N4148WT") (footprint "Diode_SMD:D_SOD-523")
+    )
+    (path "/ea7fdac0-4451-48b5-bbfd-e0f47d60ba04/f8fdf2c6-3214-46bf-8520-4b71ab9d1c2a"
+      (reference "D?") (unit 1) (value "1N4148WT") (footprint "Diode_SMD:D_SOD-523")
+    )
+    (path "/ea7fdac0-4451-48b5-bbfd-e0f47d60ba04/fd29b72a-5213-4768-a908-de9238bbe348"
       (reference "D?") (unit 1) (value "1N4148WT") (footprint "Diode_SMD:D_SOD-523")
     )
@@
       (reference "SW?") (unit 1) (value "SW_Push") (footprint "")
     )
-    (path "/0e04ce72-6533-49cc-b4b5-6fa7ba1a6887/6da45897-3798-4178-ae94-d41fac51109f"
-      (reference "U?") (unit 1) (value "KA78M05_TO252") (footprint "Package_TO_SOT_SMD:TO-252-2")
-    )
     (path "/0e04ce72-6533-49cc-b4b5-6fa7ba1a6887/b78937a8-6a0d-4f12-a5b8-a9031e3b41b1"

Commit message: reorganised the schematic
Parts:
- added P? (x2): USB_C_Plug, symbol Connector:USB_C_Plug
Connections:
- new net GND: P?.A1 (GND), P?.A1 (GND), P?.A12 (GND), P?.A12 (GND), P?.B1 (GND), P?.B1 (GND), P?.B12 (GND), P?.B12 (GND)
- new net MCU_Battery/USBUFPD+: P?.A6 (D+)
- new net MCU_Battery/USBUFPD-: P?.A7 (D-)
- new net MCU_Battery/VBUSIN: P?.A4 (VBUS), P?.A9 (VBUS), P?.B4 (VBUS), P?.B9 (VBUS)
- new net MCU_Battery/VBUSOUT: P?.A4 (VBUS), P?.A9 (VBUS), P?.B4 (VBUS), P?.B9 (VBUS)
Other:
- sheet MCU_Battery ports: added USBUFPD+, USBUFPD-, VBUSIN, VBUSOUT; removed none
