File: KeyboardPCB/Key_Array.kicad_sch (KiCad schematic)
At the start: 0 parts

Commit message: keyboard added
Parts:
- added D? (x23): 1N4148WT, Diode_SMD:D_SOD-523, symbol Diode:1N4148WT
Connections:
- new net IROW0: D?.1 (K), D?.1 (K), D?.1 (K), D?.1 (K), D?.1 (K), D?.1 (K), D?.1 (K), D?.1 (K), D?.1 (K), D?.1 (K), D?.1 (K)
- new net IROW1: D?.1 (K), D?.1 (K), D?.1 (K), D?.1 (K), D?.1 (K), D?.1 (K), D?.1 (K), D?.1 (K)
- new net IROW2: D?.1 (K)
- new net IROW3: D?.1 (K)
- new net IROW4: D?.1 (K), D?.1 (K)

Commit message: added some diodes
Parts:
- added D? (x7): 1N4148WT, Diode_SMD:D_SOD-523, symbol Diode:1N4148WT
Connections:
- net IROW2: now also D?.1 (K), D?.1 (K), D?.1 (K), D?.1 (K), D?.1 (K), D?.1 (K)
- net IROW3: now also D?.1 (K)

Commit message: Equipment added
Parts:
- gave numbers to parts that had none: 30
Changed lines of the file:
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@@
+    (stroke (width 0) (type default) (color 0 0 0 0))
+  )
+  (wire (pts (xy 38.1 25.4) (xy 38.1 152.4))
     (stroke (width 0) (type default) (color 0 0 0 0))
   )
@@
   )
   (wire (pts (xy 101.6 25.4) (xy 101.6 152.4))
-    (stroke (width 0) (type default) (color 0 0 0 0))
-  )
-  (wire (pts (xy 38.1 25.4) (xy 38.1 152.4))
     (stroke (width 0) (type default) (color 0 0 0 0))
   )
@@
   (symbol (lib_id "Diode:1N4148WT") (at 78.74 59.69 90) (unit 1)
     (in_bom yes) (on_board yes) (fields_autoplaced)
-    (property "Reference" "D?" (id 0) (at 81.28 58.4199 90)
+    (property "Reference" "D20" (id 0) (at 81.28 58.4199 90)
       (effects (font (size 1.27 1.27)) (justify right))
     )
@@
   (symbol (lib_id "Diode:1N4148WT") (at 66.04 59.69 90) (unit 1)
     (in_bom yes) (on_board yes) (fields_autoplaced)
-    (property "Reference" "D?" (id 0) (at 68.58 58.4199 90)
+    (property "Reference" "D17" (id 0) (at 68.58 58.4199 90)
       (effects (font (size 1.27 1.27)) (justify right))
     )
@@
   (symbol (lib_id "Diode:1N4148WT") (at 91.44 34.29 90) (unit 1)
     (in_bom yes) (on_board yes) (fields_autoplaced)
-    (property "Reference" "D?" (id 0) (at 93.98 33.0199 90)
+    (property "Reference" "D22" (id 0) (at 93.98 33.0199 90)
       (effects (font (size 1.27 1.27)) (justify right))
     )
@@
   (symbol (lib_id "Diode:1N4148WT") (at 53.34 34.29 90) (unit 1)
     (in_bom yes) (on_board yes) (fields_autoplaced)
-    (property "Reference" "D?" (id 0) (at 55.88 33.0199 90)
+    (property "Reference" "D13" (id 0) (at 55.88 33.0199 90)
       (effects (font (size 1.27 1.27)) (justify right))
     )
@@
   (symbol (lib_id "Diode:1N4148WT") (at 104.14 59.69 90) (unit 1)
     (in_bom yes) (on_board yes) (fields_autoplaced)
-    (property "Reference" "D?" (id 0) (at 106.68 58.4199 90)
+    (property "Reference" "D26" (id 0) (at 106.68 58.4199 90)
       (effects (font (size 1.27 1.27)) (justify right))
     )
@@
   (symbol (lib_id "Diode:1N4148WT") (at 91.44 59.69 90) (unit 1)
     (in_bom yes) (on_board yes) (fields_autoplaced)
-    (property "Reference" "D?" (id 0) (at 93.98 58.4199 90)
+    (property "Reference" "D23" (id 0) (at 93.98 58.4199 90)
       (effects (font (size 1.27 1.27)) (justify right))
     )
@@
   (symbol (lib_id "Diode:1N4148WT") (at 78.74 85.09 90) (unit 1)
     (in_bom yes) (on_board yes) (fields_autoplaced)
-    (property "Reference" "D?" (id 0) (at 81.28 83.8199 90)
+    (property "Reference" "D21" (id 0) (at 81.28 83.8199 90)
       (effects (font (size 1.27 1.27)) (justify right))
     )
@@
   (symbol (lib_id "Diode:1N4148WT") (at 129.54 34.29 90) (unit 1)
     (in_bom yes) (on_board yes) (fields_autoplaced)
-    (property "Reference" "D?" (id 0) (at 132.08 33.0199 90)
+    (property "Reference" "D30" (id 0) (at 132.08 33.0199 90)
       (effects (font (size 1.27 1.27)) (justify right))
     )
@@
   (symbol (lib_id "Diode:1N4148WT") (at 27.94 34.29 90) (unit 1)
     (in_bom yes) (on_board yes) (fields_autoplaced)
-    (property "Reference" "D?" (id 0) (at 30.48 33.0199 90)
+    (property "Reference" "D3" (id 0) (at 30.48 33.0199 90)
       (effects (font (size 1.27 1.27)) (justify right))
     )
@@
   (symbol (lib_id "Diode:1N4148WT") (at 104.14 85.09 90) (unit 1)
     (in_bom yes) (on_board yes) (fields_autoplaced)
-    (property "Reference" "D?" (id 0) (at 106.68 83.8199 90)
+    (property "Reference" "D27" (id 0) (at 106.68 83.8199 90)
       (effects (font (size 1.27 1.27)) (justify right))
     )
@@
   (symbol (lib_id "Diode:1N4148WT") (at 116.84 34.29 90) (unit 1)
     (in_bom yes) (on_board yes) (fields_autoplaced)
-    (property "Reference" "D?" (id 0) (at 119.38 33.0199 90)
+    (property "Reference" "D28" (id 0) (at 119.38 33.0199 90)
       (effects (font (size 1.27 1.27)) (justify right))
     )
@@
   (symbol (lib_id "Diode:1N4148WT") (at 66.04 34.29 90) (unit 1)
     (in_bom yes) (on_board yes) (fields_autoplaced)
-    (property "Reference" "D?" (id 0) (at 68.58 33.0199 90)
+    (property "Reference" "D16" (id 0) (at 68.58 33.0199 90)
       (effects (font (size 1.27 1.27)) (justify right))
     )
@@
   (symbol (lib_id "Diode:1N4148WT") (at 53.34 59.69 90) (unit 1)
     (in_bom yes) (on_board yes) (fields_autoplaced)
-    (property "Reference" "D?" (id 0) (at 55.88 58.4199 90)
+    (property "Reference" "D14" (id 0) (at 55.88 58.4199 90)
       (effects (font (size 1.27 1.27)) (justify right))
     )
@@
   (symbol (lib_id "Diode:1N4148WT") (at 154.94 34.29 90) (unit 1)
     (in_bom yes) (on_board yes) (fields_autoplaced)
-    (property "Reference" "D?" (id 0) (at 157.48 33.0199 90)
+    (property "Reference" "D32" (id 0) (at 157.48 33.0199 90)
       (effects (font (size 1.27 1.27)) (justify right))
     )
@@
   (symbol (lib_id "Diode:1N4148WT") (at 142.24 34.29 90) (unit 1)
     (in_bom yes) (on_board yes) (fields_autoplaced)
-    (property "Reference" "D?" (id 0) (at 144.78 33.0199 90)
+    (property "Reference" "D31" (id 0) (at 144.78 33.0199 90)
       (effects (font (size 1.27 1.27)) (justify right))
     )
@@
   (symbol (lib_id "Diode:1N4148WT") (at 40.64 59.69 90) (unit 1)
     (in_bom yes) (on_board yes) (fields_autoplaced)
-    (property "Reference" "D?" (id 0) (at 43.18 58.4199 90)
+    (property "Reference" "D9" (id 0) (at 43.18 58.4199 90)
       (effects (font (size 1.27 1.27)) (justify right))
     )
@@
   (symbol (lib_id "Diode:1N4148WT") (at 53.34 85.09 90) (unit 1)
     (in_bom yes) (on_board yes) (fields_autoplaced)
-    (property "Reference" "D?" (id 0) (at 55.88 83.8199 90)
+    (property "Reference" "D15" (id 0) (at 55.88 83.8199 90)
       (effects (font (size 1.27 1.27)) (justify right))
     )
@@
   (symbol (lib_id "Diode:1N4148WT") (at 40.64 135.89 90) (unit 1)
     (in_bom yes) (on_board yes) (fields_autoplaced)
-    (property "Reference" "D?" (id 0) (at 43.18 134.6199 90)
+    (property "Reference" "D12" (id 0) (at 43.18 134.6199 90)
       (effects (font (size 1.27 1.27)) (justify right))
     )
@@
   (symbol (lib_id "Diode:1N4148WT") (at 27.94 85.09 90) (unit 1)
     (in_bom yes) (on_board yes) (fields_autoplaced)
-    (property "Reference" "D?" (id 0) (at 30.48 83.8199 90)
+    (property "Reference" "D5" (id 0) (at 30.48 83.8199 90)
       (effects (font (size 1.27 1.27)) (justify right))
     )
@@
   (symbol (lib_id "Diode:1N4148WT") (at 91.44 85.09 90) (unit 1)
     (in_bom yes) (on_board yes) (fields_autoplaced)
-    (property "Reference" "D?" (id 0) (at 93.98 83.8199 90)
+    (property "Reference" "D24" (id 0) (at 93.98 83.8199 90)
       (effects (font (size 1.27 1.27)) (justify right))
     )
@@
   (symbol (lib_id "Diode:1N4148WT") (at 78.74 34.29 90) (unit 1)
     (in_bom yes) (on_board yes) (fields_autoplaced)
-    (property "Reference" "D?" (id 0) (at 81.28 33.0199 90)
+    (property "Reference" "D19" (id 0) (at 81.28 33.0199 90)
       (effects (font (size 1.27 1.27)) (justify right))
     )
@@
   (symbol (lib_id "Diode:1N4148WT") (at 66.04 85.09 90) (unit 1)
     (in_bom yes) (on_board yes) (fields_autoplaced)
-    (property "Reference" "D?" (id 0) (at 68.58 83.8199 90)
+    (property "Reference" "D18" (id 0) (at 68.58 83.8199 90)
       (effects (font (size 1.27 1.27)) (justify right))
     )
@@
   (symbol (lib_id "Diode:1N4148WT") (at 40.64 34.29 90) (unit 1)
     (in_bom yes) (on_board yes) (fields_autoplaced)
-    (property "Reference" "D?" (id 0) (at 43.18 33.0199 90)
+    (property "Reference" "D8" (id 0) (at 43.18 33.0199 90)
       (effects (font (size 1.27 1.27)) (justify right))
     )
@@
   (symbol (lib_id "Diode:1N4148WT") (at 104.14 34.29 90) (unit 1)
     (in_bom yes) (on_board yes) (fields_autoplaced)
-    (property "Reference" "D?" (id 0) (at 106.68 33.0199 90)
+    (property "Reference" "D25" (id 0) (at 106.68 33.0199 90)
       (effects (font (size 1.27 1.27)) (justify right))
     )
@@
   (symbol (lib_id "Diode:1N4148WT") (at 116.84 59.69 90) (unit 1)
     (in_bom yes) (on_board yes) (fields_autoplaced)
-    (property "Reference" "D?" (id 0) (at 119.38 58.4199 90)
+    (property "Reference" "D29" (id 0) (at 119.38 58.4199 90)
       (effects (font (size 1.27 1.27)) (justify right))
     )
@@
   (symbol (lib_id "Diode:1N4148WT") (at 27.94 59.69 90) (unit 1)
     (in_bom yes) (on_board yes) (fields_autoplaced)
-    (property "Reference" "D?" (id 0) (at 30.48 58.4199 90)
+    (property "Reference" "D4" (id 0) (at 30.48 58.4199 90)
       (effects (font (size 1.27 1.27)) (justify right))
     )
@@
   (symbol (lib_id "Diode:1N4148WT") (at 27.94 110.49 90) (unit 1)
     (in_bom yes) (on_board yes) (fields_autoplaced)
-    (property "Reference" "D?" (id 0) (at 30.48 109.2199 90)
+    (property "Reference" "D6" (id 0) (at 30.48 109.2199 90)
       (effects (font (size 1.27 1.27)) (justify right))
     )
@@
   (symbol (lib_id "Diode:1N4148WT") (at 27.94 135.89 90) (unit 1)
     (in_bom yes) (on_board yes) (fields_autoplaced)
-    (property "Reference" "D?" (id 0) (at 30.48 134.6199 90)
+    (property "Reference" "D7" (id 0) (at 30.48 134.6199 90)
       (effects (font (size 1.27 1.27)) (justify right))
     )
@@
   (symbol (lib_id "Diode:1N4148WT") (at 40.64 110.49 90) (unit 1)
     (in_bom yes) (on_board yes) (fields_autoplaced)
-    (property "Reference" "D?" (id 0) (at 43.18 109.2199 90)
+    (property "Reference" "D11" (id 0) (at 43.18 109.2199 90)
       (effects (font (size 1.27 1.27)) (justify right))
     )
@@
   (symbol (lib_id "Diode:1N4148WT") (at 40.64 85.09 90) (unit 1)
     (in_bom yes) (on_board yes) (fields_autoplaced)
-    (property "Reference" "D?" (id 0) (at 43.18 83.8199 90)
-      (effects (font (size 1.27 1.27)) (justify right))
-    )
+    (property "Reference" "D10" (id 0) (at 43.18 83.8199 90)
+      (effects (font (size 1.27 1.27)) (justify right))
+    )

Commit message: Added more devices.
Parts:
- added D33, D34, D35, D36, D37: 1N4148WT, Diode_SMD:D_SOD-523, symbol Diode:1N4148WT
- added S10: MX_N8, TS18525SL160SMTTR, symbol keyboard_syms:TS18-5-25-SL-160-SMT-TR
- added S11: MX_N9, TS18525SL160SMTTR, symbol keyboard_syms:TS18-5-25-SL-160-SMT-TR
- added S12: MX_N0, TS18525SL160SMTTR, symbol keyboard_syms:TS18-5-25-SL-160-SMT-TR
- added S13: MX_TAB1, TS18525SL160SMTTR, symbol keyboard_syms:TS18-5-25-SL-160-SMT-TR
- added S14: MX_CAPS1, TS18525SL160SMTTR, symbol keyboard_syms:TS18-5-25-SL-160-SMT-TR
- added S15: MX_LSHIFT, TS18525SL160SMTTR, symbol keyboard_syms:TS18-5-25-SL-160-SMT-TR
- added S16: MX_LCTRL1, TS18525SL160SMTTR, symbol keyboard_syms:TS18-5-25-SL-160-SMT-TR
- added S17: MX_Q1, TS18525SL160SMTTR, symbol keyboard_syms:TS18-5-25-SL-160-SMT-TR
- added S18: MX_A1, TS18525SL160SMTTR, symbol keyboard_syms:TS18-5-25-SL-160-SMT-TR
- added S19: MX_\, TS18525SL160SMTTR, symbol keyboard_syms:TS18-5-25-SL-160-SMT-TR
- added S2, S3: MX_N1, TS18525SL160SMTTR, symbol keyboard_syms:TS18-5-25-SL-160-SMT-TR
- added S20: MX_LWIN1, TS18525SL160SMTTR, symbol keyboard_syms:TS18-5-25-SL-160-SMT-TR
- added S21: MX_W1, TS18525SL160SMTTR, symbol keyboard_syms:TS18-5-25-SL-160-SMT-TR
- added S22: MX_S1, TS18525SL160SMTTR, symbol keyboard_syms:TS18-5-25-SL-160-SMT-TR
- added S23: MX_E1, TS18525SL160SMTTR, symbol keyboard_syms:TS18-5-25-SL-160-SMT-TR
- added S24: MX_D1, TS18525SL160SMTTR, symbol keyboard_syms:TS18-5-25-SL-160-SMT-TR
- added S25: MX_R1, TS18525SL160SMTTR, symbol keyboard_syms:TS18-5-25-SL-160-SMT-TR
- added S26: MX_F1, TS18525SL160SMTTR, symbol keyboard_syms:TS18-5-25-SL-160-SMT-TR
- added S27: MX_T1, TS18525SL160SMTTR, symbol keyboard_syms:TS18-5-25-SL-160-SMT-TR
- added S28: MX_G1, TS18525SL160SMTTR, symbol keyboard_syms:TS18-5-25-SL-160-SMT-TR
- added S29: MX_Y1, TS18525SL160SMTTR, symbol keyboard_syms:TS18-5-25-SL-160-SMT-TR
- added S30: MX_H1, TS18525SL160SMTTR, symbol keyboard_syms:TS18-5-25-SL-160-SMT-TR
- added S31: MX_U1, TS18525SL160SMTTR, symbol keyboard_syms:TS18-5-25-SL-160-SMT-TR
- added S32: MX_I1, TS18525SL160SMTTR, symbol keyboard_syms:TS18-5-25-SL-160-SMT-TR
- added S33: MX_-1, TS18525SL160SMTTR, symbol keyboard_syms:TS18-5-25-SL-160-SMT-TR
- added S34: MX_=1, TS18525SL160SMTTR, symbol keyboard_syms:TS18-5-25-SL-160-SMT-TR
- added S35: MX_BKSPC1, TS18525SL160SMTTR, symbol keyboard_syms:TS18-5-25-SL-160-SMT-TR
- added S36: MX_DEL1, TS18525SL160SMTTR, symbol keyboard_syms:TS18-5-25-SL-160-SMT-TR
- added S4: MX_N2, TS18525SL160SMTTR, symbol keyboard_syms:TS18-5-25-SL-160-SMT-TR
- added S5: MX_N3, TS18525SL160SMTTR, symbol keyboard_syms:TS18-5-25-SL-160-SMT-TR
- added S6: MX_N4, TS18525SL160SMTTR, symbol keyboard_syms:TS18-5-25-SL-160-SMT-TR
- added S7: MX_N5, TS18525SL160SMTTR, symbol keyboard_syms:TS18-5-25-SL-160-SMT-TR
- added S8: MX_N6, TS18525SL160SMTTR, symbol keyboard_syms:TS18-5-25-SL-160-SMT-TR
- added S9: MX_N7, TS18525SL160SMTTR, symbol keyboard_syms:TS18-5-25-SL-160-SMT-TR
Connections:
- net ICOL0: now also S13.2 (N2), S14.2 (N2), S15.2 (N2), S16.2 (N2), S2.2 (N2)
- net ICOL1: now also S17.2 (N2), S18.2 (N2), S19.2 (N2), S20.2 (N2), S3.2 (N2)
- net ICOL10: now also S12.2 (N2)
- net ICOL11: now also S33.2 (N2)
- net ICOL12: now also S34.2 (N2)
- net ICOL13: now also S35.2 (N2)
- net ICOL14: now also S36.2 (N2)
- net ICOL2: now also S21.2 (N2), S22.2 (N2), S4.2 (N2)
- net ICOL3: now also S23.2 (N2), S24.2 (N2), S5.2 (N2)
- net ICOL4: now also S25.2 (N2), S26.2 (N2), S6.2 (N2)
- net ICOL5: now also S27.2 (N2), S28.2 (N2), S7.2 (N2)
- net ICOL6: now also S29.2 (N2), S30.2 (N2), S8.2 (N2)
- net ICOL7: now also S31.2 (N2), S9.2 (N2)
- net ICOL8: now also S10.2 (N2), S32.2 (N2)
- net ICOL9: now also S11.2 (N2)
- net IROW0: now also D34.1 (K), D35.1 (K), D36.1 (K), D37.1 (K)
- net IROW1: now also D33.1 (K)
- net at D20.2 (A): now also S25.3 (C1)
- net at D17.2 (A): now also S23.3 (C1)
- net at D22.2 (A): now also S7.3 (C1)
- net at D13.2 (A): now also S4.3 (C1)
- net at D26.2 (A): now also S29.3 (C1)
- net at D23.2 (A): now also S27.3 (C1)
- net at D21.2 (A): now also S26.3 (C1)
- net at D30.2 (A): now also S10.3 (C1)
- net at D3.2 (A): now also S2.3 (C1)
- net at D27.2 (A): now also S30.3 (C1)
- net at D28.2 (A): now also S9.3 (C1)
- net at D16.2 (A): now also S5.3 (C1)
- net at D14.2 (A): now also S21.3 (C1)
- net at D32.2 (A): now also S12.3 (C1)
- net at D31.2 (A): now also S11.3 (C1)
- net at D9.2 (A): now also S17.3 (C1)
- net at D15.2 (A): now also S22.3 (C1)
- net at D12.2 (A): now also S20.3 (C1)
- net at D5.2 (A): now also S14.3 (C1)
- net at D24.2 (A): now also S28.3 (C1)
- net at D19.2 (A): now also S6.3 (C1)
- net at D18.2 (A): now also S24.3 (C1)
- net at D8.2 (A): now also S3.3 (C1)
- net at D25.2 (A): now also S8.3 (C1)
- net at D29.2 (A): now also S31.3 (C1)
- net at D4.2 (A): now also S13.3 (C1)
- net at D6.2 (A): now also S15.3 (C1)
- net at D7.2 (A): now also S16.3 (C1)
- net at D11.2 (A): now also S19.3 (C1)
- net at D10.2 (A): now also S18.3 (C1)
- new net: D36.2 (A), S35.3 (C1)
- new net: D37.2 (A), S36.3 (C1)
- new net: D33.2 (A), S32.3 (C1)
- new net: D34.2 (A), S33.3 (C1)
- new net: D35.2 (A), S34.3 (C1)
